File: RP2040 GPS.kicad_sch (KiCad schematic)
At the start: 7 parts, among them SW1 PB NO, SW2 DPDT

Commit message: Layout Update
Parts:
- removed RP1: Adafruit_Feather_RP2040, symbol MCU_Module:Adafruit_Feather_RP2040
- added MCU1: Adafruit_Feather_RP2040, symbol MCU_Module:Adafruit_Feather_RP2040
- SW1: value PB NO -> RESET
Connections:
- net at GPS1.1 (SDA): now also MCU1.17 (SDA)
- net at GPS1.3 (TX): now also MCU1.14 (RX)
- net at GPS1.4 (RX): now also MCU1.15 (TX)
- net at GPS1.6 (SCL): now also MCU1.18 (SCL)
- net at SW1.2: now also MCU1.1 (RST)
- net at OLED1.1 (VCC): now also GPS1.5 (VCC), MCU1.2 (3.3V)
- net at OLED1.3 (DIN): now also MCU1.12 (MO)
- net at OLED1.4 (CLK): now also MCU1.11 (SCK)
- net at OLED1.6 (DC): now also MCU1.9 (24)
- net at OLED1.7 (RST): now also MCU1.16 (D4)
- net at R1.2, R2.1: now also MCU1.5 (A0)
- net at SW2.5 (B): now also MCU1.27 (EN)
- net at SW2.2 (B): now also MCU1.28 (VBAT)
- net Earth: no longer names the net of GPS1.2 (GND), OLED1.2 (GND), R1.1, SW1.1, SW2.6 (C)
- net Earth: now also MCU1.4 (GND); no longer GPS1.5 (VCC)
Other:
- title: Feather RP2040 GPS -> Adafruit Feather RP2040 GPS
- moved on the sheet: GPS1, R2, SW2
